File: drivers.kicad_sch (KiCad schematic)
At the start: 16 parts, among them J1 Conn_01x04_Pin, U2 TMC2209-LA

Commit message: PCB schematic design
Parts:
- removed R9: 6k8, symbol Device:R_Small
- added C19, C22, C24, C26, C29, C30: 100n, symbol Device:C
- added C20, C27: 100n, symbol Device:C_Small
- added C21, C28: 100u, symbol Device:C_Polarized
- added C25, C31: 22n, symbol Device:C_Small
- added R15, R17, R20, R22: 10k, symbol Device:R_Small
- added R16, R21, R7: 1k, symbol Device:R_Small
- added R18, R19, R23, R24: 220m, symbol Device:R_Small
- added U4, U5: TMC2209-LA, Package_DFN_QFN:VQFN-28-1EP_5x5mm_P0.5mm_EP3.7x3.7mm, symbol Driver_Motor:TMC2209-LA
- R13, R14: value 150m -> 220m
- R6: value 56k -> 1k
Connections:
- net +3.3V: now also C19.2, C26.2, R15.2, R17.2, R20.2, R22.2, U4.15 (VCC_IO), U4.9 (MS1/AD0), U5.15 (VCC_IO), U5.9 (MS1/AD0); no longer R6.2
- net GND: now also C19.1, C21.2, C22.2, C24.2, C26.1, C28.2, C29.2, C30.2, R18.1, R19.2, R23.1, R24.2, U4.10 (MS2/AD1), U4.13 (CLK), U4.18 (GND), U4.20 (STDBY), U4.29 (GND), U4.3 (GND), U5.10 (MS2/AD1), U5.13 (CLK), U5.18 (GND), U5.20 (STDBY), U5.29 (GND), U5.3 (GND); no longer U2.7 (SPREAD)
- net VM: now also C20.2, C21.1, C22.1, C24.1, C27.2, C28.1, C29.1, C30.1, U4.22 (VS), U4.28 (VS), U5.22 (VS), U5.28 (VS)
- net at R6.1: now also U4.16 (STEP); no longer U2.17 (VREF)
- new net: C31.1, U5.5 (CPI)
- new net: C31.2, U5.4 (CPO)
- new net: R19.1, U4.27 (BRB)
- new net: R20.1, U5.2 (~{EN})
- new net: R22.1, U5.11 (DIAG)
- new net: R23.2, U5.23 (BRA)
- new net: R16.1, U4.14 (~{PD}/UART)
- new net: R21.1, U5.14 (~{PD}/UART)
- new net: R24.1, U5.27 (BRB)
- new net: R7.1, U5.16 (STEP)
- new net: C27.1, U5.6 (VCP)
- new net: C25.1, U4.5 (CPI)
- new net: C25.2, U4.4 (CPO)
- new net: R17.1, U4.11 (DIAG)
- new net: R15.1, U4.2 (~{EN})
- new net: R18.2, U4.23 (BRA)
- new net: C20.1, U4.6 (VCP)
- new net DIR2: U4.19 (DIR)
- new net DIR3: U5.19 (DIR)
- new net M2_A+: U4.24 (OA1)
- new net M2_A-: U4.21 (OA2)
- new net M2_B+: U4.26 (OB1)
- new net M2_B-: U4.1 (OB2)
- new net M3_A+: U5.24 (OA1)
- new net M3_A-: U5.21 (OA2)
- new net M3_B+: U5.26 (OB1)
- new net M3_B-: U5.1 (OB2)
- new net RX2: R16.2
- new net RX3: R21.2
- new net STEP2: R6.2
- new net STEP3: R7.2
- no-connect marks 3 -> 12
Other:
- moved on the sheet: J1

Commit message: Finished design
Parts:
- C16: renamed from C21; footprint (none) -> Capacitor_THT:CP_Radial_D5.0mm_P2.00mm
- C17: renamed from C28; footprint (none) -> Capacitor_THT:CP_Radial_D5.0mm_P2.00mm
- C18: renamed from C10; footprint (none) -> Capacitor_THT:CP_Radial_D5.0mm_P2.00mm
- C19: renamed from C22; footprint (none) -> Capacitor_SMD:C_0603_1608Metric_Pad1.08x0.95mm_HandSolder
- C20: renamed from C29; footprint (none) -> Capacitor_SMD:C_0603_1608Metric_Pad1.08x0.95mm_HandSolder
- C21: renamed from C12; footprint (none) -> Capacitor_SMD:C_0603_1608Metric_Pad1.08x0.95mm_HandSolder
- C22: renamed from C24; footprint (none) -> Capacitor_SMD:C_0603_1608Metric_Pad1.08x0.95mm_HandSolder
- C23: renamed from C30; footprint (none) -> Capacitor_SMD:C_0603_1608Metric_Pad1.08x0.95mm_HandSolder
- C24: renamed from C15; footprint (none) -> Capacitor_SMD:C_0603_1608Metric_Pad1.08x0.95mm_HandSolder
- C25: renamed from C19; footprint (none) -> Capacitor_SMD:C_0603_1608Metric_Pad1.08x0.95mm_HandSolder
- C26: renamed from C20; footprint (none) -> Capacitor_SMD:C_0603_1608Metric_Pad1.08x0.95mm_HandSolder
- C27: renamed from C26; footprint (none) -> Capacitor_SMD:C_0603_1608Metric_Pad1.08x0.95mm_HandSolder
- C28: renamed from C17; footprint (none) -> Capacitor_SMD:C_0603_1608Metric_Pad1.08x0.95mm_HandSolder
- C29: renamed from C27; footprint (none) -> Capacitor_SMD:C_0603_1608Metric_Pad1.08x0.95mm_HandSolder
- C30: renamed from C18; footprint (none) -> Capacitor_SMD:C_0603_1608Metric_Pad1.08x0.95mm_HandSolder
- C31: renamed from C25; footprint (none) -> Capacitor_SMD:C_0603_1608Metric_Pad1.08x0.95mm_HandSolder
- C32: renamed from C31; footprint (none) -> Capacitor_SMD:C_0603_1608Metric_Pad1.08x0.95mm_HandSolder
- C33: renamed from C23; footprint (none) -> Capacitor_SMD:C_0603_1608Metric_Pad1.08x0.95mm_HandSolder
- J6: renamed from J1; footprint (none) -> Connector_PinHeader_2.54mm:PinHeader_1x04_P2.54mm_Vertical
- R16: renamed from R6; footprint (none) -> Resistor_SMD:R_0603_1608Metric_Pad0.98x0.95mm_HandSolder
- R17: renamed from R7; footprint (none) -> Resistor_SMD:R_0603_1608Metric_Pad0.98x0.95mm_HandSolder
- R18: renamed from R5; footprint (none) -> Resistor_SMD:R_0603_1608Metric_Pad0.98x0.95mm_HandSolder
- R19: renamed from R16; footprint (none) -> Resistor_SMD:R_0603_1608Metric_Pad0.98x0.95mm_HandSolder
- R20: renamed from R21; footprint (none) -> Resistor_SMD:R_0603_1608Metric_Pad0.98x0.95mm_HandSolder
- R21: renamed from R10; footprint (none) -> Resistor_SMD:R_0603_1608Metric_Pad0.98x0.95mm_HandSolder
- R22: renamed from R15; footprint (none) -> Resistor_SMD:R_0603_1608Metric_Pad0.98x0.95mm_HandSolder
- R23: renamed from R20; footprint (none) -> Resistor_SMD:R_0603_1608Metric_Pad0.98x0.95mm_HandSolder
- R24: renamed from R11; footprint (none) -> Resistor_SMD:R_0603_1608Metric_Pad0.98x0.95mm_HandSolder
- R25: renamed from R17; footprint (none) -> Resistor_SMD:R_0603_1608Metric_Pad0.98x0.95mm_HandSolder
- R26: renamed from R18; footprint (none) -> Resistor_SMD:R_0603_1608Metric_Pad0.98x0.95mm_HandSolder
- R27: renamed from R22; footprint (none) -> Resistor_SMD:R_0603_1608Metric_Pad0.98x0.95mm_HandSolder
- R28: renamed from R23; footprint (none) -> Resistor_SMD:R_0603_1608Metric_Pad0.98x0.95mm_HandSolder
- R29: renamed from R12; footprint (none) -> Resistor_SMD:R_0603_1608Metric_Pad0.98x0.95mm_HandSolder
- R30: renamed from R13; footprint (none) -> Resistor_SMD:R_0603_1608Metric_Pad0.98x0.95mm_HandSolder
- R31: renamed from R19; footprint (none) -> Resistor_SMD:R_0603_1608Metric_Pad0.98x0.95mm_HandSolder
- R32: renamed from R24; footprint (none) -> Resistor_SMD:R_0603_1608Metric_Pad0.98x0.95mm_HandSolder
- R33: renamed from R14; footprint (none) -> Resistor_SMD:R_0603_1608Metric_Pad0.98x0.95mm_HandSolder
- renumbered U4 to U6, U5 to U7, U2 to U8
Connections:
- net GND: now also U6.7 (SPREAD), U7.7 (SPREAD), U8.7 (SPREAD)
- net A4988_DIR: now reaches J6.3 (Pin_3)
- net A4988_STEP: now reaches J6.4 (Pin_4)
Other:
- moved on the sheet: J6

Commit message: Started troublefixing
Parts:
- removed R19, R20: 1k, Resistor_SMD:R_0603_1608Metric_Pad0.98x0.95mm_HandSolder, symbol Device:R_Small
- added R23, R24: 1k, Resistor_SMD:R_0603_1608Metric_Pad0.98x0.95mm_HandSolder, symbol Device:R_Small
- renumbered C16 to C18, C17 to C19, C18 to C20, C19 to C21, C20 to C22, C21 to C23, C22 to C24, C23 to C25, C24 to C26, C25 to C27, C26 to C28, C27 to C29, C28 to C30, C29 to C31, C30 to C32, C31 to C33, C32 to C34, C33 to C35, R16 to R20, R17 to R21, R18 to R22, R21 to R25, R22 to R26, R23 to R27, R24 to R28, R25 to R29, R26 to R30, R27 to R31, R28 to R32, R29 to R33, R30 to R34, R31 to R35, R32 to R36, R33 to R37
Connections:
- net RX1: now also U8.14 (~{PD}/UART)
- net RX2: now also U6.14 (~{PD}/UART), R23.2
- net RX3: now also U7.14 (~{PD}/UART), R24.2
- net TX1: now reaches R25.1
- net TX1: no longer U8.14 (~{PD}/UART)
- new net TX2: R23.1
- new net TX3: R24.1
Other:
- moved on the sheet: R25

Commit message: Corrected wrong footprints
Parts:
- R30, R32, R35, R36, R37: footprint Resistor_SMD:R_0603_1608Metric_Pad0.98x0.95mm_HandSolder -> Resistor_SMD:R_2512_6332Metric_Pad1.40x3.35mm_HandSolder
Changed lines of the file:
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@@
 			)
 		)
-		(property "Footprint" "Resistor_SMD:R_0603_1608Metric_Pad0.98x0.95mm_HandSolder"
+		(property "Footprint" "Resistor_SMD:R_2512_6332Metric_Pad1.40x3.35mm_HandSolder"
 			(at 170.18 102.87 0)
 			(hide yes)
@@
 			)
 		)
-		(property "Footprint" "Resistor_SMD:R_0603_1608Metric_Pad0.98x0.95mm_HandSolder"
+		(property "Footprint" "Resistor_SMD:R_2512_6332Metric_Pad1.40x3.35mm_HandSolder"
 			(at 254 101.6 0)
 			(hide yes)
@@
 			)
 		)
-		(property "Footprint" "Resistor_SMD:R_0603_1608Metric_Pad0.98x0.95mm_HandSolder"
+		(property "Footprint" "Resistor_SMD:R_2512_6332Metric_Pad1.40x3.35mm_HandSolder"
 			(at 254 104.14 0)
 			(hide yes)
@@
 			)
 		)
-		(property "Footprint" "Resistor_SMD:R_0603_1608Metric_Pad0.98x0.95mm_HandSolder"
+		(property "Footprint" "Resistor_SMD:R_2512_6332Metric_Pad1.40x3.35mm_HandSolder"
 			(at 86.36 105.41 0)
 			(hide yes)
@@
 			)
 		)
-		(property "Footprint" "Resistor_SMD:R_0603_1608Metric_Pad0.98x0.95mm_HandSolder"
+		(property "Footprint" "Resistor_SMD:R_2512_6332Metric_Pad1.40x3.35mm_HandSolder"
 			(at 170.18 100.33 0)
 			(hide yes)

Commit message: Started rerouting changes
Parts:
- R30: renamed from R34; footprint Resistor_SMD:R_0603_1608Metric_Pad0.98x0.95mm_HandSolder -> Resistor_SMD:R_2512_6332Metric_Pad1.40x3.35mm_HandSolder
- renumbered C18 to C16, C19 to C17, C20 to C18, C21 to C19, C22 to C20, C26 to C21, C24 to C22, C25 to C23, C23 to C24, C27 to C25, C28 to C26, C29 to C27, C30 to C28, C31 to C29, C32 to C30, C33 to C31, C34 to C32, C35 to C33, R20 to R16, R21 to R17, R22 to R18, R23 to R19, R24 to R20, R25 to R21, R26 to R22, R27 to R23, R28 to R24, R29 to R25, R30 to R26, R31 to R27, R32 to R28, R33 to R29, R35 to R31, R36 to R32, R37 to R33
