File: power.kicad_sch (KiCad schematic)
At the start: 15 parts, among them U14 TPS2121RUXR, U3 LMR51430

Commit message: PCB schematic design
Parts:
- added BT1: Battery, Connector_JST:JST_XH_B2B-XH-A_1x02_P2.50mm_Vertical, symbol Device:Battery
- added C33: 100n, symbol Device:C
- added D2: SS34, Diode_SMD:D_SMA_Handsoldering, symbol Diode:SS34
- added L2: 47u, Inductor_SMD:L_12x12mm_H8mm, symbol Device:L
- added R42: 10m, symbol Device:R
- added R8: 2k8, symbol Device:R
- added R9: 330, symbol Device:R
- added U17: INA219BxDCN, Package_TO_SOT_SMD:SOT-23-8, symbol Sensor_Energy:INA219BxDCN
- added VR1: XL6009, Project_Components:DPAK170P1435X465-6N, symbol Project_Components:XL6009
Connections:
- net +BATT: now also L2.1, R42.1, U17.1 (IN+), VR1.2 (EN), VR1.4 (VIN)
- net GND: now also R9.2, VR1.1 (GND)
- new net: D2.2 (A), L2.2, R8.1, VR1.3 (SW), VR1.6 (SW)
- new net: BT1.1 (+), R42.2, U17.2 (IN-)
- new net: R8.2, R9.1, VR1.5 (FB)
- new net +3.3V_1: C33.2, U17.4 (VS)
- new net GND_1: BT1.2 (-), C33.1, U17.3 (GND), U17.7 (A0), U17.8 (A1)
- new net INA_SCL: U17.5 (SCL)
- new net INA_SDA: U17.6 (SDA)
- new net VM: D2.1 (K)

Commit message: Finished design
Parts:
- removed C57: 47n, symbol Device:C_Small
- removed D3: RED, symbol Device:LED
- removed R29: 270k, symbol Device:R_Small
- removed R30: 100k, symbol Device:R_Small
- removed R32: 10k, symbol Device:R_Small
- removed R34: 120, symbol Device:R
- removed U14: TPS2121RUXR, TPS2121RUXR:IC_TPS2121RUXR, symbol TPS2121RUXR:TPS2121RUXR
- added C14: 1u, Capacitor_SMD:C_0603_1608Metric_Pad1.08x0.95mm_HandSolder, symbol Device:C_Small
- added D2: RED, LED_SMD:LED_0603_1608Metric_Pad1.05x0.95mm_HandSolder, symbol Device:LED
- added R10: 21k5, Resistor_SMD:R_0603_1608Metric_Pad0.98x0.95mm_HandSolder, symbol Device:R_Small
- added R3: 120, Resistor_SMD:R_0603_1608Metric_Pad0.98x0.95mm_HandSolder, symbol Device:R
- added R4: 7k, Resistor_SMD:R_0603_1608Metric_Pad0.98x0.95mm_HandSolder, symbol Device:R_Small
- added R6, R9: 5k, Resistor_SMD:R_0603_1608Metric_Pad0.98x0.95mm_HandSolder, symbol Device:R_Small
- added R7: 12k, Resistor_SMD:R_0603_1608Metric_Pad0.98x0.95mm_HandSolder, symbol Device:R_Small
- added U3: TPS2121RUXR, TPS2121RUXR:IC_TPS2121RUXR, symbol Project_Components:TPS2121RUXR
- C10: renamed from C11; footprint (none) -> Capacitor_SMD:C_0603_1608Metric_Pad1.08x0.95mm_HandSolder
- C11: renamed from C13; footprint (none) -> Capacitor_SMD:C_0603_1608Metric_Pad1.08x0.95mm_HandSolder
- C12: renamed from C14; footprint (none) -> Capacitor_SMD:C_0603_1608Metric_Pad1.08x0.95mm_HandSolder
- C13: renamed from C16; footprint (none) -> Capacitor_SMD:C_0603_1608Metric_Pad1.08x0.95mm_HandSolder
- C15: renamed from C33; footprint (none) -> Capacitor_SMD:C_0603_1608Metric_Pad1.08x0.95mm_HandSolder
- L1: footprint (none) -> Project_Components:WE-XHMI_4040
- L2: footprint Inductor_SMD:L_12x12mm_H8mm -> Inductor_SMD:L_Changjiang_FXL1365
- R11: renamed from R42; footprint (none) -> Resistor_SMD:R_0603_1608Metric_Pad0.98x0.95mm_HandSolder
- R12: renamed from R8; footprint (none) -> Resistor_SMD:R_0603_1608Metric_Pad0.98x0.95mm_HandSolder
- R13: renamed from R9; footprint (none) -> Resistor_SMD:R_0603_1608Metric_Pad0.98x0.95mm_HandSolder
- R5: renamed from R3; footprint (none) -> Resistor_SMD:R_0603_1608Metric_Pad0.98x0.95mm_HandSolder
- R8: renamed from R4; footprint (none) -> Resistor_SMD:R_0603_1608Metric_Pad0.98x0.95mm_HandSolder
- U2: renamed from U3; value LMR51430 -> LMR51420
- renumbered D2 to D3, U17 to U4
Connections:
- net +3.3V_1 is gone; now on net +3.3V: C15.2, U4.4 (VS)
- net GND_1 is gone; now on net GND: BT1.2 (-), C15.1, U4.3 (GND), U4.7 (A0), U4.8 (A1)
- net +3.3V: now also R3.1
- net +BATT: now also R7.1, U3.2 (IN2), U3.2_1 (IN2)
- net GND: now also C14.2, R10.2, R6.2, R9.2, U3.12 (GND), U3.4 (OV2), U3.5 (OV1)
- net POWER_STATE: now also D2.1 (K), U3.9 (ST)
- net VBUS: now also R4.1, U3.7 (IN1), U3.7_1 (IN1)
- net at C11.1, C12.1, U2.3 (VIN)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: now also U3.1 (OUT), U3.1_1 (OUT), U3.8 (OUT), U3.8_1 (OUT)
- new net: C14.1, U3.11 (SS)
- new net: R7.2, R9.1, U3.3 (CP2)
- new net: R10.1, U3.10 (ILIM)
- new net: R4.2, R6.1, U3.6 (PR1)
- new net: D2.2 (A), R3.2
Other:
- moved on the sheet: D3, L2, R12, R13, VR1

Commit message: Final tweaks
Parts:
- R4: value 7k -> 47k
- R6, R9: value 5k -> 33k
- R7: value 12k -> 82k
Changed lines of the file:
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@@
 			)
 		)
-		(property "Value" "12k"
+		(property "Value" "82k"
 			(at 48.26 86.3599 0)
 			(show_name no)
@@
 			)
 		)
-		(property "Value" "5k"
+		(property "Value" "33k"
 			(at 29.21 83.8199 0)
 			(show_name no)
@@
 			)
 		)
-		(property "Value" "5k"
+		(property "Value" "33k"
 			(at 48.26 95.2499 0)
 			(show_name no)
@@
 			)
 		)
-		(property "Value" "7k"
+		(property "Value" "47k"
 			(at 29.21 76.1999 0)
 			(show_name no)

Commit message: Final tweaks
Parts:
- added C34: 100u, Capacitor_THT:CP_Radial_D5.0mm_P2.00mm, symbol Device:C_Polarized
- added C35: 100n, Capacitor_SMD:C_0603_1608Metric_Pad1.08x0.95mm_HandSolder, symbol Device:C
Connections:
- net GND: now also C34.2, C35.1
- net at BT1.1 (+), R11.2, U4.2 (IN-): now also C34.1, C35.2
Other:
- moved on the sheet: BT1, C15, R11, U4

Commit message: Minor tweaks
Changed lines of the file:
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@@
-	)
-	(junction
-		(at 135.89 71.12)
-		(diameter 0)
-		(color 0 0 0 0)
 	)
 	(junction
@@
 	(wire
 		(pts
-			(xy 135.89 71.12) (xy 147.32 71.12)
+			(xy 95.25 71.12) (xy 147.32 71.12)
 		)
 		(stroke
@@
 		(pts
 			(xy 62.23 189.23) (xy 71.12 189.23)
-		)
-		(stroke
-			(width 0)
-			(type default)
-		)
-	)
-	(wire
-		(pts
-			(xy 95.25 71.12) (xy 135.89 71.12)
 		)
 		(stroke
@@
 					(unit 1)
 				)
-			)
-		)
-	)
-	(symbol
-		(lib_id "power:PWR_FLAG")
-		(at 135.89 71.12 0)
-		(unit 1)
-		(body_style 1)
-		(exclude_from_sim no)
-		(in_bom yes)
-		(on_board yes)
-		(in_pos_files yes)
-		(dnp no)
-		(fields_autoplaced yes)
-		(property "Reference" "#FLG01"
-			(at 135.89 69.215 0)
-			(hide yes)
-			(show_name no)
-			(do_not_autoplace no)
-			(effects
-				(font
-					(size 1.27 1.27)
-				)
-			)
-		)
-		(property "Value" "PWR_FLAG"
-			(at 135.89 66.04 0)
-			(show_name no)
-			(do_not_autoplace no)
-			(effects
-				(font
-					(size 1.27 1.27)
-				)
-			)
-		)
-		(property "Footprint" ""
-			(at 135.89 71.12 0)
-			(hide yes)
-			(show_name no)
-			(do_not_autoplace no)
-			(effects
-				(font
-					(size 1.27 1.27)
-				)
-			)
-		)
-		(property "Datasheet" ""
-			(at 135.89 71.12 0)
-			(hide yes)
-			(show_name no)
-			(do_not_autoplace no)
-			(effects
-				(font
-					(size 1.27 1.27)
-				)
-			)
-		)
-		(property "Description" "Special symbol for telling ERC where power comes from"
-			(at 135.89 71.12 0)
-			(hide yes)
-			(show_name no)
-			(do_not_autoplace no)
-			(effects
-				(font
-					(size 1.27 1.27)
-				)
-			)
-		)
-		(pin "1"
-		)
-		(instances
-			(project "Orion"
-				(path "/f9e05184-c88b-4a88-ae9c-ab2bdb32be7c/c5103ceb-5325-4a84-a025-9638a412984e/236a6b28-69fd-491e-8932-30aa549da18f"
-					(reference "#FLG01")
-					(unit 1)
-				)

Commit message: Started troublefixing
Parts:
- renumbered C35 to C16, C34 to C17, R6 to R10, R7 to R11, R8 to R12, R9 to R13, R10 to R14, R11 to R15, R12 to R16, R13 to R17, R3 to R7, R4 to R8, R5 to R9

Commit message: Corrected wrong footprints
Parts:
- R15: footprint Resistor_SMD:R_0603_1608Metric_Pad0.98x0.95mm_HandSolder -> Resistor_SMD:R_0805_2012Metric_Pad1.20x1.40mm_HandSolder
Changed lines of the file:
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@@
 			)
 		)
-		(property "Footprint" "Resistor_SMD:R_0603_1608Metric_Pad0.98x0.95mm_HandSolder"
+		(property "Footprint" "Resistor_SMD:R_0805_2012Metric_Pad1.20x1.40mm_HandSolder"
 			(at 191.262 118.11 90)
 			(hide yes)

Commit message: Started rerouting changes
Parts:
- renumbered C17 to C34, C16 to C35, R14 to R10, R15 to R11, R16 to R12, R17 to R13, R7 to R3, R8 to R4, R9 to R5, R10 to R6, R11 to R7, R12 to R8, R13 to R9
Changed lines of the file:
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@@
 		(dnp no)
 		(fields_autoplaced yes)
-		(property "Reference" "R15"
+		(property "Reference" "R11"
 			(at 195.58 116.8399 0)
 			(show_name no)
@@
 			(project "Orion"
 				(path "/f9e05184-c88b-4a88-ae9c-ab2bdb32be7c/c5103ceb-5325-4a84-a025-9638a412984e/236a6b28-69fd-491e-8932-30aa549da18f"
-					(reference "R15")
+					(reference "R11")
 					(unit 1)
 				)
@@
 		(dnp no)
 		(fields_autoplaced yes)
-		(property "Reference" "R17"
+		(property "Reference" "R13"
 			(at 73.66 181.6099 0)
 			(show_name no)
@@
 			(project "Orion"
 				(path "/f9e05184-c88b-4a88-ae9c-ab2bdb32be7c/c5103ceb-5325-4a84-a025-9638a412984e/236a6b28-69fd-491e-8932-30aa549da18f"
-					(reference "R17")
+					(reference "R13")
 					(unit 1)
 				)
@@
 		(in_pos_files yes)
 		(dnp no)
-		(property "Reference" "R11"
+		(property "Reference" "R7"
 			(at 48.26 83.8199 0)
 			(show_name no)
@@
 			(project "Orion"
 				(path "/f9e05184-c88b-4a88-ae9c-ab2bdb32be7c/c5103ceb-5325-4a84-a025-9638a412984e/236a6b28-69fd-491e-8932-30aa549da18f"
-					(reference "R11")
+					(reference "R7")
 					(unit 1)
 				)
@@
 		(dnp no)
 		(fields_autoplaced yes)
-		(property "Reference" "R16"
+		(property "Reference" "R12"
 			(at 73.66 171.4499 0)
 			(show_name no)
@@
 			(project "Orion"
 				(path "/f9e05184-c88b-4a88-ae9c-ab2bdb32be7c/c5103ceb-5325-4a84-a025-9638a412984e/236a6b28-69fd-491e-8932-30aa549da18f"
-					(reference "R16")
+					(reference "R12")
 					(unit 1)
 				)
@@
 		(in_pos_files yes)
 		(dnp no)
-		(property "Reference" "C17"
+		(property "Reference" "C34"
 			(at 182.88 141.986 90)
 			(show_name no)
@@
 			(project "Orion"
 				(path "/f9e05184-c88b-4a88-ae9c-ab2bdb32be7c/c5103ceb-5325-4a84-a025-9638a412984e/236a6b28-69fd-491e-8932-30aa549da18f"
-					(reference "C17")
+					(reference "C34")
 					(unit 1)
 				)
@@
 		(in_pos_files yes)
 		(dnp no)
-		(property "Reference" "R14"
+		(property "Reference" "R10"
 			(at 69.342 100.838 0)
 			(show_name no)
@@
 			(project "Orion"
 				(path "/f9e05184-c88b-4a88-ae9c-ab2bdb32be7c/c5103ceb-5325-4a84-a025-9638a412984e/236a6b28-69fd-491e-8932-30aa549da18f"
-					(reference "R14")
+					(reference "R10")
 					(unit 1)
 				)
@@
 		(in_pos_files yes)
 		(dnp no)
-		(property "Reference" "R12"
+		(property "Reference" "R8"
 			(at 232.41 83.8199 0)
 			(show_name no)
@@
 			(project "Orion"
 				(path "/f9e05184-c88b-4a88-ae9c-ab2bdb32be7c/c5103ceb-5325-4a84-a025-9638a412984e/236a6b28-69fd-491e-8932-30aa549da18f"
-					(reference "R12")
+					(reference "R8")
 					(unit 1)
 				)
@@
 		(in_pos_files yes)
 		(dnp no)
-		(property "Reference" "R10"
+		(property "Reference" "R6"
 			(at 29.21 81.2799 0)
 			(show_name no)
@@
 			(project "Orion"
 				(path "/f9e05184-c88b-4a88-ae9c-ab2bdb32be7c/c5103ceb-5325-4a84-a025-9638a412984e/236a6b28-69fd-491e-8932-30aa549da18f"
-					(reference "R10")
+					(reference "R6")
 					(unit 1)
 				)
@@
 		(in_pos_files yes)
 		(dnp no)
-		(property "Reference" "R13"
+		(property "Reference" "R9"
 			(at 48.26 92.7099 0)
 			(show_name no)
@@
 			(project "Orion"
 				(path "/f9e05184-c88b-4a88-ae9c-ab2bdb32be7c/c5103ceb-5325-4a84-a025-9638a412984e/236a6b28-69fd-491e-8932-30aa549da18f"
-					(reference "R13")
+					(reference "R9")
 					(unit 1)
 				)
@@
 		(in_pos_files yes)
 		(dnp no)
-		(property "Reference" "C16"
+		(property "Reference" "C35"
 			(at 184.15 126.492 90)
 			(show_name no)
@@
 			(project "Orion"
 				(path "/f9e05184-c88b-4a88-ae9c-ab2bdb32be7c/c5103ceb-5325-4a84-a025-9638a412984e/236a6b28-69fd-491e-8932-30aa549da18f"
-					(reference "C16")
+					(reference "C35")
 					(unit 1)
 				)
@@
 		(in_pos_files yes)
 		(dnp no)
-		(property "Reference" "R8"
+		(property "Reference" "R4"
 			(at 29.21 73.6599 0)
 			(show_name no)
@@
 			(project "Orion"
 				(path "/f9e05184-c88b-4a88-ae9c-ab2bdb32be7c/c5103ceb-5325-4a84-a025-9638a412984e/236a6b28-69fd-491e-8932-30aa549da18f"
-					(reference "R8")
+					(reference "R4")
 					(unit 1)
 				)
@@
 		(dnp no)
 		(fields_autoplaced yes)
-		(property "Reference" "R7"
+		(property "Reference" "R3"
 			(at 83.82 53.34 90)
 			(show_name no)
@@
 			(project "Orion"
 				(path "/f9e05184-c88b-4a88-ae9c-ab2bdb32be7c/c5103ceb-5325-4a84-a025-9638a412984e/236a6b28-69fd-491e-8932-30aa549da18f"
-					(reference "R7")
+					(reference "R3")
 					(unit 1)
 				)
@@
 		(in_pos_files yes)
 		(dnp no)
-		(property "Reference" "R9"
+		(property "Reference" "R5"
 			(at 232.41 76.1999 0)
 			(show_name no)
@@
 			(project "Orion"
 				(path "/f9e05184-c88b-4a88-ae9c-ab2bdb32be7c/c5103ceb-5325-4a84-a025-9638a412984e/236a6b28-69fd-491e-8932-30aa549da18f"
-					(reference "R9")
+					(reference "R5")
 					(unit 1)
 				)
