File: Orion.kicad_pcb (KiCad board)
At the start: 6 copper layers, 0 parts

Commit message: Finished design
Parts:
- added BT1: Battery, Connector_JST:JST_XH_B2B-XH-A_1x02_P2.50mm_Vertical, F.Cu at (114.7, 101.1)
- added C1: 100u, Capacitor_SMD:C_0603_1608Metric_Pad1.08x0.95mm_HandSolder, F.Cu at (112.0, 36.0)
- added C10: 100n, Capacitor_SMD:C_0603_1608Metric_Pad1.08x0.95mm_HandSolder, F.Cu at (118.2, 80.3)
- added C11: 1u, Capacitor_SMD:C_0603_1608Metric_Pad1.08x0.95mm_HandSolder, F.Cu at (116.9, 87.4)
- added C12: 100n, Capacitor_SMD:C_0603_1608Metric_Pad1.08x0.95mm_HandSolder, F.Cu at (116.9, 85.8)
- added C13: 47u, Capacitor_SMD:C_0603_1608Metric_Pad1.08x0.95mm_HandSolder, F.Cu at (112.6, 78.5)
- added C14: 1u, Capacitor_SMD:C_0603_1608Metric_Pad1.08x0.95mm_HandSolder, F.Cu at (125.7, 85.6)
- added C15: 100n, Capacitor_SMD:C_0603_1608Metric_Pad1.08x0.95mm_HandSolder, F.Cu at (117.1, 93.9)
- added C16: 100u, Capacitor_THT:CP_Radial_D5.0mm_P2.00mm, F.Cu at (93.3, 66.4)
- added C17: 100u, Capacitor_THT:CP_Radial_D5.0mm_P2.00mm, F.Cu at (93.2, 80.5)
- added C18: 100u, Capacitor_THT:CP_Radial_D5.0mm_P2.00mm, F.Cu at (93.3, 52.3)
- added C19: 100n, Capacitor_SMD:C_0603_1608Metric_Pad1.08x0.95mm_HandSolder, F.Cu at (86.4, 67.4)
- added C2: 22p, Capacitor_SMD:C_0603_1608Metric_Pad1.08x0.95mm_HandSolder, F.Cu at (110.5, 36.0)
- added C20: 100n, Capacitor_SMD:C_0603_1608Metric_Pad1.08x0.95mm_HandSolder, F.Cu at (88.1, 81.4)
- added C21: 100n, Capacitor_SMD:C_0603_1608Metric_Pad1.08x0.95mm_HandSolder, F.Cu at (86.4, 53.3)
- added C22: 100n, Capacitor_SMD:C_0603_1608Metric_Pad1.08x0.95mm_HandSolder, F.Cu at (88.2, 67.4)
- added C23: 100n, Capacitor_SMD:C_0603_1608Metric_Pad1.08x0.95mm_HandSolder, F.Cu at (86.3, 81.4)
- added C24: 100n, Capacitor_SMD:C_0603_1608Metric_Pad1.08x0.95mm_HandSolder, F.Cu at (88.2, 53.3)
- added C25: 100n, Capacitor_SMD:C_0603_1608Metric_Pad1.08x0.95mm_HandSolder, F.Cu at (75.9, 66.6)
- added C26: 100n, Capacitor_SMD:C_0603_1608Metric_Pad1.08x0.95mm_HandSolder, F.Cu at (84.6, 60.4)
- added C27: 100n, Capacitor_SMD:C_0603_1608Metric_Pad1.08x0.95mm_HandSolder, F.Cu at (75.9, 80.6)
- added C28: 100n, Capacitor_SMD:C_0603_1608Metric_Pad1.08x0.95mm_HandSolder, F.Cu at (75.9, 52.5)
- added C29: 100n, Capacitor_SMD:C_0603_1608Metric_Pad1.08x0.95mm_HandSolder, F.Cu at (84.5, 74.5)
- added C3: 100u, Capacitor_SMD:C_0603_1608Metric_Pad1.08x0.95mm_HandSolder, F.Cu at (108.9, 36.0)
- added C30: 100n, Capacitor_SMD:C_0603_1608Metric_Pad1.08x0.95mm_HandSolder, F.Cu at (84.6, 46.4)
- added C31: 22n, Capacitor_SMD:C_0603_1608Metric_Pad1.08x0.95mm_HandSolder, F.Cu at (80.6, 59.3)
- added C32: 22n, Capacitor_SMD:C_0603_1608Metric_Pad1.08x0.95mm_HandSolder, F.Cu at (80.5, 73.4)
- added C33: 22n, Capacitor_SMD:C_0603_1608Metric_Pad1.08x0.95mm_HandSolder, F.Cu at (80.6, 45.3)
- added C4: 22u, Capacitor_SMD:C_0603_1608Metric_Pad1.08x0.95mm_HandSolder, F.Cu at (107.3, 36.0)
- added C5: 100u, Capacitor_SMD:C_0603_1608Metric_Pad1.08x0.95mm_HandSolder, F.Cu at (105.7, 36.0)
- added C6: 100n, Capacitor_SMD:C_0603_1608Metric_Pad1.08x0.95mm_HandSolder, F.Cu at (104.1, 36.0)
- added C7: 10u, Capacitor_SMD:C_0603_1608Metric_Pad1.08x0.95mm_HandSolder, F.Cu at (100.8, 37.7)
- added C8: 100n, Capacitor_SMD:C_0603_1608Metric_Pad1.08x0.95mm_HandSolder, F.Cu at (99.2, 37.7)
- added C9: 100n, Capacitor_SMD:C_0603_1608Metric_Pad1.08x0.95mm_HandSolder, F.Cu at (141.0, 37.5)
- added D1: RED, LED_SMD:LED_0603_1608Metric_Pad1.05x0.95mm_HandSolder, F.Cu at (138.2, 36.6)
- added D2: RED, LED_SMD:LED_0603_1608Metric_Pad1.05x0.95mm_HandSolder, F.Cu at (129.7, 88.1)
- added D3: SS34, Diode_SMD:D_SMA_Handsoldering, F.Cu at (99.3, 85.4)
- added FB1: LI0603G121R-10, Inductor_SMD:L_0603_1608Metric_Pad1.05x0.95mm_HandSolder, F.Cu at (126.9, 99.8)
- added H1: MountingHole_Pad, MountingHole:MountingHole_3.2mm_M3_DIN965_Pad, F.Cu at (70.1, 100.4)
- added H2: MountingHole_Pad, MountingHole:MountingHole_3.2mm_M3_DIN965_Pad, F.Cu at (68.8, 38.7)
- added H3: MountingHole_Pad, MountingHole:MountingHole_3.2mm_M3_DIN965_Pad, F.Cu at (132.3, 67.6)
- added H4: MountingHole_Pad, MountingHole:MountingHole_3.2mm_M3_DIN965_Pad, F.Cu at (146.3, 99.7)
- added J1: Conn_01x04_Pin, Connector_PinHeader_2.54mm:PinHeader_1x04_P2.54mm_Vertical, F.Cu at (148.0, 42.2)
- added J2: USB4105GFA, Project_Components:GCT_USB4105GFA, F.Cu at (133.0, 103.7)
- added J3: Conn_01x04_Pin, Connector_JST:JST_XH_B4B-XH-A_1x04_P2.50mm_Vertical, F.Cu at (67.5, 53.8)
- added J4: Conn_01x04_Pin, Connector_JST:JST_XH_B4B-XH-A_1x04_P2.50mm_Vertical, F.Cu at (67.5, 67.8)
- added J5: Conn_01x04_Pin, Connector_JST:JST_XH_B4B-XH-A_1x04_P2.50mm_Vertical, F.Cu at (67.5, 81.9)
- added J6: Conn_01x04_Pin, Connector_PinHeader_2.54mm:PinHeader_1x04_P2.54mm_Vertical, F.Cu at (148.0, 54.6)
- added L1: 5u6, Project_Components:WE-XHMI_4040, F.Cu at (111.7, 81.8)
- added L2: 47u, Inductor_SMD:L_Changjiang_FXL1365, F.Cu at (103.9, 97.9)
- added R1: 120, Resistor_SMD:R_0603_1608Metric_Pad0.98x0.95mm_HandSolder, F.Cu at (134.6, 36.6)
- added R10: 21k5, Resistor_SMD:R_0603_1608Metric_Pad0.98x0.95mm_HandSolder, F.Cu at (127.2, 85.6)
- added R11: 10m, Resistor_SMD:R_0603_1608Metric_Pad0.98x0.95mm_HandSolder, F.Cu at (113.8, 97.0)
- added R12: 2k8, Resistor_SMD:R_0603_1608Metric_Pad0.98x0.95mm_HandSolder, F.Cu at (83.3, 101.9)
- added R13: 330, Resistor_SMD:R_0603_1608Metric_Pad0.98x0.95mm_HandSolder, F.Cu at (84.9, 101.9)
- added R14: 5k1, Resistor_SMD:R_0603_1608Metric_Pad0.98x0.95mm_HandSolder, F.Cu at (140.8, 99.8)
- added R15: 5k1, Resistor_SMD:R_0603_1608Metric_Pad0.98x0.95mm_HandSolder, F.Cu at (139.2, 99.8)
- added R16: 1k, Resistor_SMD:R_0603_1608Metric_Pad0.98x0.95mm_HandSolder, F.Cu at (78.9, 68.3)
- added R17: 1k, Resistor_SMD:R_0603_1608Metric_Pad0.98x0.95mm_HandSolder, F.Cu at (78.9, 82.3)
- added R18: 1k, Resistor_SMD:R_0603_1608Metric_Pad0.98x0.95mm_HandSolder, F.Cu at (78.9, 54.2)
- added R19: 1k, Resistor_SMD:R_0603_1608Metric_Pad0.98x0.95mm_HandSolder, F.Cu at (75.0, 62.3)
- added R2: 10k, Resistor_SMD:R_0603_1608Metric_Pad0.98x0.95mm_HandSolder, F.Cu at (102.4, 37.7)
- added R20: 1k, Resistor_SMD:R_0603_1608Metric_Pad0.98x0.95mm_HandSolder, F.Cu at (75.0, 76.4)
- added R21: 1k, Resistor_SMD:R_0603_1608Metric_Pad0.98x0.95mm_HandSolder, F.Cu at (75.0, 48.3)
- added R22: 10k, Resistor_SMD:R_0603_1608Metric_Pad0.98x0.95mm_HandSolder, F.Cu at (83.0, 58.4)
- added R23: 10k, Resistor_SMD:R_0603_1608Metric_Pad0.98x0.95mm_HandSolder, F.Cu at (83.0, 72.5)
- added R24: 10k, Resistor_SMD:R_0603_1608Metric_Pad0.98x0.95mm_HandSolder, F.Cu at (83.0, 44.4)
- added R25: 10k, Resistor_SMD:R_0603_1608Metric_Pad0.98x0.95mm_HandSolder, F.Cu at (75.9, 64.1)
- added R26: 220m, Resistor_SMD:R_0603_1608Metric_Pad0.98x0.95mm_HandSolder, F.Cu at (87.3, 64.8)
- added R27: 10k, Resistor_SMD:R_0603_1608Metric_Pad0.98x0.95mm_HandSolder, F.Cu at (75.8, 78.2)
- added R28: 220m, Resistor_SMD:R_0603_1608Metric_Pad0.98x0.95mm_HandSolder, F.Cu at (87.2, 78.8)
- added R29: 10k, Resistor_SMD:R_0603_1608Metric_Pad0.98x0.95mm_HandSolder, F.Cu at (75.9, 50.0)
- added R3: 120, Resistor_SMD:R_0603_1608Metric_Pad0.98x0.95mm_HandSolder, F.Cu at (130.6, 85.6)
- added R30: 220m, Resistor_SMD:R_0603_1608Metric_Pad0.98x0.95mm_HandSolder, F.Cu at (87.3, 50.7)
- added R31: 220m, Resistor_SMD:R_0603_1608Metric_Pad0.98x0.95mm_HandSolder, F.Cu at (87.3, 63.1)
- added R32: 220m, Resistor_SMD:R_0603_1608Metric_Pad0.98x0.95mm_HandSolder, F.Cu at (87.2, 77.2)
- added R33: 220m, Resistor_SMD:R_0603_1608Metric_Pad0.98x0.95mm_HandSolder, F.Cu at (87.3, 49.1)
- added R34: 47k, Resistor_SMD:R_0603_1608Metric_Pad0.98x0.95mm_HandSolder, F.Cu at (134.8, 40.6)
- added R35: 47k, Resistor_SMD:R_0603_1608Metric_Pad0.98x0.95mm_HandSolder, F.Cu at (134.8, 39.0)
- added R36: 47k, Resistor_SMD:R_0603_1608Metric_Pad0.98x0.95mm_HandSolder, F.Cu at (122.0, 56.2)
- added R37: 47k, Resistor_SMD:R_0603_1608Metric_Pad0.98x0.95mm_HandSolder, F.Cu at (123.6, 56.2)
- added R4: 7k, Resistor_SMD:R_0603_1608Metric_Pad0.98x0.95mm_HandSolder, F.Cu at (128.8, 90.9)
- added R5: 100k, Resistor_SMD:R_0603_1608Metric_Pad0.98x0.95mm_HandSolder, F.Cu at (120.8, 81.3)
- added R6: 5k, Resistor_SMD:R_0603_1608Metric_Pad0.98x0.95mm_HandSolder, F.Cu at (127.3, 92.8)
- added R7: 12k, Resistor_SMD:R_0603_1608Metric_Pad0.98x0.95mm_HandSolder, F.Cu at (124.2, 90.9)
- added R8: 22k1, Resistor_SMD:R_0603_1608Metric_Pad0.98x0.95mm_HandSolder, F.Cu at (120.8, 84.8)
- added R9: 5k, Resistor_SMD:R_0603_1608Metric_Pad0.98x0.95mm_HandSolder, F.Cu at (125.7, 92.8)
- added SW1: RST, Button_Switch_SMD:Panasonic_EVQPUJ_EVQPUA, F.Cu at (94.5, 37.7)
- added SW2: BOOT, Button_Switch_SMD:Panasonic_EVQPUJ_EVQPUA, F.Cu at (145.9, 37.5)
- added TP1: VBUS, TestPoint:TestPoint_Pad_D1.5mm, F.Cu at (131.2, 92.3)
- added TP2: 3V3, TestPoint:TestPoint_Pad_D1.5mm, F.Cu at (113.1, 73.9)
- added TP3: VM, TestPoint:TestPoint_Pad_D1.5mm, F.Cu at (103.8, 84.2)
- added TP4: BATT, TestPoint:TestPoint_Pad_D1.5mm, F.Cu at (109.5, 88.7)
- added TP5: GND, TestPoint:TestPoint_Pad_D1.5mm, F.Cu at (104.9, 74.0)
- added U1: ESP32-S3-WROOM-1, Project_Components:ESP32-S3-WROOM-1_novias, F.Cu at (122.8, 40.6)
- added U2: LMR51420, Package_TO_SOT_SMD:SOT-23-6_Handsoldering, F.Cu at (117.4, 83.0)
- added U3: TPS2121RUXR, TPS2121RUXR:IC_TPS2121RUXR, F.Cu at (126.5, 89.3)
- added U4: INA219BxDCN, Package_TO_SOT_SMD:SOT-23-8, F.Cu at (114.4, 93.6)
- added U5: SRV05-4, Package_TO_SOT_SMD:SOT-23-6_Handsoldering, F.Cu at (133.0, 95.6)
- added U6: TMC2209-LA, Package_DFN_QFN:VQFN-28-1EP_5x5mm_P0.5mm_EP3.7x3.7mm, F.Cu at (80.8, 64.1)
- added U7: TMC2209-LA, Package_DFN_QFN:VQFN-28-1EP_5x5mm_P0.5mm_EP3.7x3.7mm, F.Cu at (80.8, 78.2)
- added U8: TMC2209-LA, Package_DFN_QFN:VQFN-28-1EP_5x5mm_P0.5mm_EP3.7x3.7mm, F.Cu at (80.9, 50.1)
- added VR1: XL6009, Project_Components:DPAK170P1435X465-6N, F.Cu at (91.5, 95.8)
Routing:
- net +3.3V: track 0.00 -> 301.1 mm, vias 0 -> 4
- net VM: track 0.00 -> 107.3 mm, vias 0 -> 6
- net GND: track 0.00 -> 79.5 mm, vias 0 -> 108
- net /Project Architecture/Connectors/USB_D+: track 0.00 -> 63.1 mm
- net /Project Architecture/Connectors/USB_D-: track 0.00 -> 62.8 mm
- net +BATT: track 0.00 -> 61.8 mm
- net RX3: track 0.00 -> 59.9 mm, vias 0 -> 2
- net STEP3: track 0.00 -> 56.6 mm, vias 0 -> 2
- net RX2: track 0.00 -> 53.4 mm, vias 0 -> 2
- net DIR3: track 0.00 -> 52.7 mm, vias 0 -> 2
- net RX1: track 0.00 -> 51.5 mm, vias 0 -> 2
- net STEP2: track 0.00 -> 49.1 mm, vias 0 -> 2
- net /Project Architecture/MCU/INA_SCL: track 0.00 -> 48.0 mm, vias 0 -> 2
- net /Project Architecture/MCU/INA_SDA: track 0.00 -> 48.0 mm, vias 0 -> 2
- net DIR2: track 0.00 -> 46.8 mm, vias 0 -> 2
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- added copper zone on B.Cu, net GND
- added copper zone on F.Cu, net GND
- added copper zone on In1.Cu, net GND
- added copper zone on In2.Cu, net GND
Other:
- board outline added: 86.1 x 71.9 mm
- copper layers 6 -> 4
- board text removed: "${ASSEMBLY_NOTES}"
- board text removed: "${FABRICATION_NOTES}"
- board text removed: "30°"
- board text removed: "3× 120°"
- board text removed: "All dimensions are in millimeters unless otherwise specified."
- board text removed: "Bottom View"
- board text removed: "Components"
- board text removed: "Drill Table"
- board text removed: "Impedance Table"
- board text removed: "Layer Stack Legend"
- board text removed: "Top View"
- board text removed: "X"
- board text removed: "Y"

Commit message: Final tweaks
Parts:
- C1, C3, C5: footprint Capacitor_SMD:C_0603_1608Metric_Pad1.08x0.95mm_HandSolder -> Capacitor_SMD:C_1206_3216Metric_Pad1.33x1.80mm_HandSolder
- SW1, SW2: footprint Button_Switch_SMD:Panasonic_EVQPUJ_EVQPUA -> Button_Switch_SMD:SW_SPST_PTS647_Sx38
- moved C1 3.50 mm to (108.6, 36.7)
- moved C4 3.29 mm to (110.6, 35.9)
- moved C3 2.86 mm to (106.1, 36.7)
- moved SW1 2.54 mm to (92.0, 37.0)
- moved C6 2.44 mm to (101.7, 36.0)
- moved C7 2.44 mm to (98.4, 37.7)
- moved C8 2.44 mm to (96.8, 37.7)
- moved R2 2.44 mm to (100.0, 37.7)
- moved C5 2.17 mm to (103.6, 36.7)
- moved C2 1.67 mm to (112.1, 35.9)
- moved SW2 0.64 mm to (146.3, 37.0)
Routing:
- net GND: track 79.5 -> 55.7 mm, vias 108 -> 103
- net Net-(U1-EN): track 22.6 -> 25.8 mm
- net +3.3V: track 301.1 -> 302.2 mm
- net Net-(U1-IO0): track 26.6 -> 27.2 mm

Commit message: Final tweaks
Parts:
- added C34: 100u, Capacitor_THT:CP_Radial_D5.0mm_P2.00mm, F.Cu at (123.1, 99.0)
- added C35: 100n, Capacitor_SMD:C_0603_1608Metric_Pad1.08x0.95mm_HandSolder, F.Cu at (123.1, 95.4)
- R4: value 7k -> 47k
- R6, R9: value 5k -> 33k
- R7: value 12k -> 82k
Routing:
- net Net-(BT1-+): track 6.70 -> 18.6 mm
- net GND: vias 103 -> 104

Commit message: Started rerouting changes
Parts:
- R11: footprint Resistor_SMD:R_0603_1608Metric_Pad0.98x0.95mm_HandSolder -> Resistor_SMD:R_0805_2012Metric_Pad1.20x1.40mm_HandSolder
- R26, R28, R30, R31, R32, R33: footprint Resistor_SMD:R_0603_1608Metric_Pad0.98x0.95mm_HandSolder -> Resistor_SMD:R_2512_6332Metric_Pad1.40x3.35mm_HandSolder
- moved R20 46.6 mm to (116.8, 56.0)
- moved R19 37.9 mm to (108.4, 44.4)
- moved R21 34.0 mm to (108.2, 41.0), turned to 0 degrees
- moved R26 12.4 mm to (99.6, 63.2)
- moved R28 7.35 mm to (93.8, 75.6)
- moved R32 7.35 mm to (93.8, 73.9)
- moved R33 6.84 mm to (93.1, 45.4)
- moved R30 5.82 mm to (92.7, 48.6)
- moved R31 5.17 mm to (91.3, 59.8)
Connections:
- R19 pad 1: Net-(U6-~{PD}/UART) -> TX2
- R20 pad 1: Net-(U7-~{PD}/UART) -> TX3
- R21 pad 1: Net-(U8-~{PD}/UART) -> TX1
- U1 pad 15: RX3 -> TX3
- U1 pad 4: RX1 -> TX1
- U1 pad 6: STEP1 -> DIR1
- U1 pad 7: DIR1 -> STEP1
- U1 pad 8: RX2 -> TX2
- U6 pad 14: Net-(U6-~{PD}/UART) -> RX2
- U7 pad 14: Net-(U7-~{PD}/UART) -> RX3
- U8 pad 14: Net-(U8-~{PD}/UART) -> RX1
Routing:
- net Net-(U7-~{PD}/UART): track 5.19 -> 0.00 mm
- net Net-(U6-~{PD}/UART): track 5.19 -> 0.00 mm
- net RX3: track 59.9 -> 65.1 mm
- net RX2: track 53.4 -> 58.6 mm
- net Net-(U8-~{PD}/UART): track 5.19 -> 0.00 mm
- net M1_A+: track 21.9 -> 26.3 mm
- net RX1: track 51.5 -> 50.1 mm, vias 2 -> 1
- net DIR1: track 43.2 -> 44.4 mm
- net M1_A-: track 17.1 -> 18.0 mm
- net STEP1: track 45.2 -> 45.9 mm
- net GND: vias 104 -> 103

Commit message: Completed changes
Parts:
- moved R26 8.05 mm to (91.6, 62.3)
- moved R19 3.20 mm to (111.4, 45.5), turned to 0 degrees
- moved R21 3.20 mm to (111.4, 40.5)
- moved R32 2.64 mm to (91.6, 72.5)
- moved R28 2.34 mm to (91.6, 76.4)
- moved R20 2.05 mm to (114.9, 55.2)
- moved R33 1.74 mm to (91.7, 44.3)
- moved R31 1.50 mm to (91.6, 58.3)
- moved R30 1.08 mm to (91.7, 48.3)
Routing:
- net RX1: track 50.1 -> 60.1 mm, vias 1 -> 4
- net Net-(U8-BRB): track 3.09 -> 8.78 mm
- net Net-(U6-BRB): track 3.09 -> 8.73 mm
- net Net-(U7-BRB): track 3.09 -> 8.55 mm
- net M3_A+: track 21.7 -> 25.9 mm
- net M2_A+: track 21.8 -> 25.9 mm
- net TX1: track 0.00 -> 4.13 mm
- net TX2: track 0.00 -> 4.12 mm
- net RX2: track 58.6 -> 62.0 mm, vias 2 -> 4
- net Net-(U7-BRA): track 3.46 -> 6.61 mm
- net Net-(U8-BRA): track 3.46 -> 6.59 mm
- net Net-(U6-BRA): track 3.46 -> 6.58 mm
- net RX3: track 65.1 -> 67.3 mm, vias 2 -> 5
- net TX3: track 0.00 -> 2.06 mm
- net M3_A-: track 16.9 -> 17.9 mm
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- removed copper zone on In1.Cu, net GND
- removed copper zone on In2.Cu, net GND
Other:
- copper layers 4 -> 2

Commit message: Finalized design
Routing:
- net +3.3V: track 303.1 -> 304.3 mm
- net STEP2: track 49.8 -> 50.6 mm
- net GND: vias 116 -> 132

Commit message: Final layout changes
Parts:
- moved R14 13.6 mm to (127.6, 96.5)
- moved TP4 10.7 mm to (106.5, 78.4)
- moved TP3 7.30 mm to (99.4, 78.4)
- moved C35 5.97 mm to (117.5, 97.4), turned to 180 degrees
- moved TP2 5.58 mm to (109.7, 78.4)
- moved TP5 4.78 mm to (103.0, 78.4)
- moved FB1 4.22 mm to (129.5, 96.5)
- moved R15 3.70 mm to (137.5, 96.5)
- moved C13 3.18 mm to (115.5, 79.8), turned to 90 degrees
- moved C21 0.46 mm to (86.5, 53.8)
- moved C24 0.46 mm to (88.3, 53.8)
- moved TP1 0.43 mm to (130.9, 92.6)
- moved C11 0.39 mm to (117.0, 87.8)
- moved C12 0.39 mm to (117.0, 86.2)
- moved C15 0.39 mm to (117.2, 94.3)
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Routing:
- net VM: track 107.3 -> 151.7 mm, vias 6 -> 0
- net +3.3V: track 304.3 -> 287.1 mm
- net DIR3: track 53.1 -> 69.3 mm, vias 2 -> 4
- net STEP3: track 56.6 -> 71.4 mm, vias 2 -> 4
- net VBUS: track 20.1 -> 10.4 mm
- net +BATT: track 61.8 -> 71.4 mm
- net RX1: track 60.1 -> 52.5 mm, vias 4 -> 2
- net RX2: track 62.0 -> 54.7 mm, vias 4 -> 2
- net RX3: track 67.3 -> 73.2 mm, vias 5 -> 4
- net VB: track 13.3 -> 8.42 mm
- net Net-(J2-CC1): track 11.1 -> 6.41 mm
- net Net-(U1-IO0): track 27.2 -> 31.5 mm
- net DIR2: track 47.2 -> 49.8 mm
- net /Project Architecture/MCU/INA_SCL: track 48.0 -> 45.6 mm
- net DIR1: track 44.4 -> 46.5 mm
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